File: SanBan/SanBan.kicad_pcb (KiCad board)
At the start: 2 copper layers, 32 parts, among them IC1 AP64500SP-13, J1 Conn_01x12_Pin, J10 Conn_01x03_Pin, J11 Conn_01x03_Pin, J12 Conn_01x04, J13 Conn_01x04, J14 Conn_01x02, J15 Conn_01x15_Socket, J16 Conn_01x15_Socket, J17 Conn_01x15_Socket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

Commit message: SanBan Rev 1.0
Parts:
- J1, J2: footprint Connector_PinSocket_2.54mm:PinSocket_1x12_P2.54mm_Vertical -> Connector_PinSocket_2.00mm:PinSocket_1x12_P2.00mm_Vertical
- J10, J11, J6, J7, J8, J9: footprint Connector_PinHeader_2.54mm:PinHeader_1x03_P2.54mm_Horizontal -> Connector_PinHeader_2.54mm:PinHeader_1x03_P2.54mm_Vertical
- J3: footprint Connector_PinSocket_2.00mm:PinSocket_1x09_P2.00mm_Vertical -> Connector_PinSocket_2.54mm:PinSocket_1x09_P2.54mm_Vertical
- J4: footprint Connector_Wire:SolderWire-0.127sqmm_1x02_P3.7mm_D0.48mm_OD1mm -> Connector_PinHeader_2.54mm:PinHeader_1x02_P2.54mm_Horizontal; moved to B.Cu
- moved R7 128.0 mm to (185.2, 71.7), turned to 90 degrees
- moved C3 127.1 mm to (176.2, 82.4), turned to -90 degrees
- moved R6 127.0 mm to (185.2, 76.2), turned to 90 degrees
- moved J1 126.9 mm to (183.0, 98.2), turned to -90 degrees
- moved C4 125.3 mm to (172.8, 71.9), turned to 180 degrees
- moved R2 123.0 mm to (176.2, 77.9), turned to -90 degrees
- moved R1 120.0 mm to (174.0, 82.4), turned to 90 degrees
- moved C5 119.0 mm to (172.8, 74.2), turned to 180 degrees
- moved J2 118.8 mm to (188.2, 70.9)
- moved C2 115.7 mm to (165.0, 81.9), turned to 90 degrees
- moved R3 115.1 mm to (174.0, 77.9), turned to -90 degrees
- moved C1 113.2 mm to (162.5, 78.5), turned to -90 degrees
- moved C6 111.7 mm to (165.9, 85.4)
- moved R4 111.3 mm to (169.4, 73.1), turned to 90 degrees
- moved J11 106.9 mm to (140.3, 70.1), turned to -90 degrees
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Routing:
- net +5V: track 0.00 -> 141.1 mm
- net 5V_ESC: track 0.00 -> 86.5 mm, vias 0 -> 1
- net I2C_CLK: track 0.00 -> 83.2 mm
- net I2C_DATA: track 0.00 -> 81.9 mm
- net GPS_RX: track 0.00 -> 78.0 mm
- net GPS_TX: track 0.00 -> 73.7 mm
- net BT_RX: track 0.00 -> 60.3 mm, vias 0 -> 2
- net BT_TX: track 0.00 -> 56.5 mm, vias 0 -> 1
- net GND: track 0.00 -> 29.3 mm, vias 0 -> 14
- net PWM3: track 0.00 -> 28.9 mm
- net +BATT: track 0.00 -> 22.8 mm
- net PWM4: track 0.00 -> 21.0 mm
- net PWM0: track 0.00 -> 18.4 mm
- net PWM1: track 0.00 -> 16.1 mm
- net PWM5: track 0.00 -> 15.7 mm
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- added copper zone on B.Cu, net GND
- added copper zone on F.Cu, net GND
Other:
- board outline added: 80 x 37 mm
- board text added: "+"
- board text added: "+ s -"
- board text added: "-"
- board text added: "."
- board text added: "0"
- board text added: "1"
- board text added: "2"
- board text added: "3"
- board text added: "4"
- board text added: "5"
- board text added: "ARDUINO"
- board text added: "BATTERY"
- board text added: "BLUETOOTH"
- board text added: "FLIGHT CONTROLLER"
- board text added: "GPS"
- board text added: "JETSON"
- board text added: "KITE"
- board text added: "MAGNETOMETER"
- board text added: "PROJECT"
- board text added: "PWM"
- board text added: "SANBAN REV 1.0"
- board text added: "SamSun 24'"
