File: SanBan/SanBan.kicad_sch (KiCad schematic)
At the start: 3 parts, among them J1 Conn_01x12_Pin, J2 Conn_01x12_Pin, J3 Conn_01x09_Pin

Commit message: First pass - added MCU, 5V PS
Parts:
- added C1: 45u, symbol Device:C
- added C2: 100n, symbol Device:C
- added C3: 0u, symbol Device:C
- added C4: 2.7n, symbol Device:C
- added C5: 39p, symbol Device:C
- added C6, C9: 10u, symbol Device:C
- added C7, C8: 22p, symbol Device:C
- added IC1: AP64500SP-13, SOIC127P600X163-9N, symbol SanBanLibrary:AP64500SP-13
- added J10, J11, J12, J13, J6, J7, J8, J9: Conn_01x03_Pin, symbol Connector:Conn_01x03_Pin
- added J4: Conn_01x02, symbol Connector_Generic:Conn_01x02
- added J5: Conn_02x03_Top_Bottom, symbol Connector_Generic:Conn_02x03_Top_Bottom
- added L1: 3.6u, symbol Device:L
- added R1: 200k, symbol Device:R
- added R2: 115k, symbol Device:R
- added R3: 22.1k, symbol Device:R
- added R4: 15.8k, symbol Device:R
- added R5: 1k, symbol Device:R
- added SW1: SW_Push_Dual, symbol Switch:SW_Push_Dual
- added U1: ATmega328PB-A, Package_QFP:TQFP-32_7x7mm_P0.8mm, symbol MCU_Microchip_ATmega:ATmega328PB-A
- added Y1: 16M, symbol Device:Crystal
Connections:
- new net: C5.2, IC1.6 (COMP), R4.1
- new net: R5.2, SW1.1
- new net: C4.2, R4.2
- new net: C7.1, U1.7 (XTAL1/PB6), Y1.2
- new net: C2.2, IC1.8 (SW), L1.1
- new net: C3.1, IC1.5 (FB), R2.2, R3.1
- new net: C8.1, U1.8 (XTAL2/PB7), Y1.1
- new net: C2.1, IC1.1 (BST)
- new net: IC1.4 (RT/CLK), R1.1
- new net: J5.2 (Pin_2), U1.15 (PB3)
- new net: J5.6 (Pin_6), U1.16 (PB4)
- new net: J5.5 (Pin_5), U1.17 (PB5)
- new net +5V: C1.1, C3.2, C9.2, J10.3 (Pin_3), J11.3 (Pin_3), J12.3 (Pin_3), J13.3 (Pin_3), J5.3 (Pin_3), J6.3 (Pin_3), J7.3 (Pin_3), J8.3 (Pin_3), J9.3 (Pin_3), L1.2, R2.1, SW1.2, U1.18 (AVCC), U1.4 (VCC)
- new net +BATT: C6.2, IC1.2 (VIN), IC1.3 (EN), J4.2 (Pin_2)
- new net GND: C1.2, C4.1, C5.1, C6.1, C7.2, C8.2, C9.1, IC1.9 (EP), J10.1 (Pin_1), J11.1 (Pin_1), J12.1 (Pin_1), J13.1 (Pin_1), J4.1 (Pin_1), J5.1 (Pin_1), J6.1 (Pin_1), J7.1 (Pin_1), J8.1 (Pin_1), J9.1 (Pin_1), R1.2, R3.2, U1.21 (GND), U1.5 (GND)
- new net PWM0: J6.2 (Pin_2), U1.30 (PD0)
- new net PWM1: J7.2 (Pin_2), U1.31 (PD1)
- new net PWM2: J8.2 (Pin_2), U1.32 (PD2)
- new net PWM3: J9.2 (Pin_2), U1.1 (PD3)
- new net PWM4: J10.2 (Pin_2), U1.9 (PD5)
- new net PWM5: J11.2 (Pin_2), U1.10 (PD6)
- new net PWM6: J12.2 (Pin_2), U1.13 (PB1)
- new net PWM7: J13.2 (Pin_2), U1.14 (PB2)
- new net RST: J5.4 (Pin_4), R5.1, U1.29 (~{RESET}/PC6)
- no-connect marks 0 -> 2
Other:
- note added: "---PROJECT KITE--- "SANBAN" FC STACK DAUGHTERBOARD PWM, POWER SUPPLY, FC BREAKOUT"
- note added: "0"
- note added: "AP64500SP-13 CIRCUIT +22.2V -> +5.0V DC-DC BUCK STEP DOWN"
- note added: "ATMEGA328PB-A CIRCUIT PWM GENERATION"
- note added: "BATTERY REGULATION"
- note added: "DAUGHTERBOARD MCU"
- note added: "DUPONT 01X03 PINS SERVOS, LEDS"
- note added: "FEB 5, 2024"
- note added: "PWM OUT"
- note added: "SANBAN"
- moved on the sheet: J1, J2, J3

Commit message: Round 2 added FC pinouts
Parts:
- added J14: Conn_01x02, symbol Connector_Generic:Conn_01x02
Connections:
- net +5V: now also J14.2 (Pin_2)
- net GND: now also IC1.7 (GND), J1.10 (Pin_10), J1.3 (Pin_3), J2.1 (Pin_1), J2.12 (Pin_12), J3.4 (Pin_4), J3.5 (Pin_5), J14.1 (Pin_1)
- net WBCM_VID: now reaches J1.1 (Pin_1)
- net WBCM_VCC: now reaches J1.2 (Pin_2)
- net DIST_BAT: now reaches J1.9 (Pin_9)
- net VTLM_VID: now reaches J2.10 (Pin_10)
- net VTLM_VCC: now reaches J2.11 (Pin_11)
- net GPS_5V: now reaches J2.2 (Pin_2)
- net GPS_RX1: now reaches J2.3 (Pin_3)
- net GPS_TX1: now reaches J2.4 (Pin_4)
- net GPS_RX3: now reaches J2.5 (Pin_5)
- net GPS_TX3: now reaches J2.6 (Pin_6)
- net VTLM_RX: now reaches J2.9 (Pin_9)
- no-connect marks 2 -> 32
Other:
- note added: "3V"
- note added: "5V"
- note added: "<|"
- note added: "BAT"
- note added: "BZ+"
- note added: "BZ-"
- note added: "CUR"
- note added: "FC BOARD PIN FOOTPRINTS UNPOPULATED"
- note added: "FC BREAKOUT"
- note added: "G"
- note added: "GND"
- note added: "LED"
- note added: "M1"
- note added: "M2"
- note added: "M3"
- note added: "M4"
- note added: "M5"
- note added: "M6"
- note added: "PROG PINS"
- note added: "RST BTN"
- note added: "RX1"
- note added: "RX3"
- note added: "RX6"
- note added: "TO BATTERY"
- note added: "TO JETSON"
- note added: "TX1"
- note added: "TX3"
- note added: "TX6"
- note added: "V0"
- note added: "VIN"
- moved on the sheet: C1, C2, C3, C4, C5, C6, IC1, J1, J10, J11, J12, J13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

Commit message: Started PCB layout
Parts:
- removed C7, C8: 22p, symbol Device:C
- removed C9: 10u, symbol Device:C
- removed J12, J13: Conn_01x03_Pin, symbol Connector:Conn_01x03_Pin
- removed J5: Conn_02x03_Top_Bottom, symbol Connector_Generic:Conn_02x03_Top_Bottom
- removed R5: 1k, symbol Device:R
- removed SW1: SW_Push_Dual, symbol Switch:SW_Push_Dual
- removed U1: ATmega328PB-A, Package_QFP:TQFP-32_7x7mm_P0.8mm, symbol MCU_Microchip_ATmega:ATmega328PB-A
- removed Y1: 16M, symbol Device:Crystal
- added J12, J13, J5: Conn_01x04, Connector_JST:JST_EH_B4B-EH-A_1x04_P2.50mm_Vertical, symbol Connector_Generic:Conn_01x04
- added J15, J16, J17, J18: Conn_01x15_Socket, Connector_PinSocket_2.54mm:PinSocket_1x15_P2.54mm_Vertical, symbol Connector:Conn_01x15_Socket
- added R6: 1K, Capacitor_SMD:C_0805_2012Metric_Pad1.18x1.45mm_HandSolder, symbol Device:R
- added R7: 2K, Capacitor_SMD:C_0805_2012Metric_Pad1.18x1.45mm_HandSolder, symbol Device:R
- C1, C2, C3, C4, C5, C6, R1, R2, R3, R4: footprint (none) -> Capacitor_SMD:C_0805_2012Metric_Pad1.18x1.45mm_HandSolder
- IC1: footprint SOIC127P600X163-9N -> SanBanLibrary:SOIC127P600X163-9N
- J1, J2: footprint (none) -> Connector_PinSocket_2.54mm:PinSocket_1x12_P2.54mm_Vertical
- J10, J11, J6, J7, J8, J9: footprint (none) -> Connector_PinHeader_2.54mm:PinHeader_1x03_P2.54mm_Horizontal
- J14: footprint (none) -> Connector_JST:JST_EH_B2B-EH-A_1x02_P2.50mm_Vertical
- J3: footprint (none) -> Connector_PinSocket_2.00mm:PinSocket_1x09_P2.00mm_Vertical
- J4: footprint (none) -> Connector_Wire:SolderWire-0.127sqmm_1x02_P3.7mm_D0.48mm_OD1mm
- L1: footprint (none) -> Inductor_SMD:L_TDK_VLS6045EX_VLS6045AF
Connections:
- net +5V: now also J15.12 (Pin_12), J17.12 (Pin_12)
- net GND: now also J12.1 (Pin_1), J13.1 (Pin_1), J15.14 (Pin_14), J17.14 (Pin_14), J5.1 (Pin_1), R7.2; no longer J1.10 (Pin_10), J1.3 (Pin_3), J2.12 (Pin_12)
- net PWM0: now also J16.6 (Pin_6), J18.6 (Pin_6)
- net PWM1: now also J16.8 (Pin_8), J18.8 (Pin_8)
- net PWM2: now also J16.9 (Pin_9), J18.9 (Pin_9)
- net PWM3: now also J16.12 (Pin_12), J18.12 (Pin_12)
- net PWM4: now also J16.13 (Pin_13), J18.13 (Pin_13)
- net PWM5: now also J16.14 (Pin_14), J18.14 (Pin_14)
- net GPS_TX: now reaches J3.1 (Pin_1)
- net GPS_TX: now also J13.3 (Pin_3)
- net GPS_RX: now reaches J3.2 (Pin_2)
- net GPS_RX: now also J13.2 (Pin_2)
- net 5V_ESC: now reaches J3.6 (Pin_6)
- net 5V_ESC: now also J12.4 (Pin_4), J13.4 (Pin_4), J5.4 (Pin_4)
- net DIST_BAT: no longer names the net of J1.9 (Pin_9)
- net GPS_5V: no longer names the net of J2.2 (Pin_2)
- net GPS_RX1 renamed BT_TX
- net BT_TX: now also J5.3 (Pin_3)
- net GPS_RX3 renamed I2C_DATA
- net I2C_DATA: now also J12.3 (Pin_3), J15.8 (Pin_8), J17.8 (Pin_8)
- net GPS_TX1: no longer names the net of J2.4 (Pin_4)
- net GPS_TX1: now also R6.1
- net GPS_TX3 renamed I2C_CLK
- net I2C_CLK: now also J12.2 (Pin_2), J15.9 (Pin_9), J17.9 (Pin_9)
- net VTLM_RX: no longer names the net of J2.9 (Pin_9)
- net VTLM_VCC: no longer names the net of J2.11 (Pin_11)
- net VTLM_VID: no longer names the net of J2.10 (Pin_10)
- net WBCM_VCC: no longer names the net of J1.2 (Pin_2)
- net WBCM_VID: no longer names the net of J1.1 (Pin_1)
- new net: J15.1 (Pin_1), J17.1 (Pin_1)
- new net: J15.10 (Pin_10), J17.10 (Pin_10)
- new net: J15.11 (Pin_11), J17.11 (Pin_11)
- new net: J15.13 (Pin_13), J17.13 (Pin_13)
- new net: J15.15 (Pin_15), J17.15 (Pin_15)
- new net: J15.2 (Pin_2), J17.2 (Pin_2)
- new net: J15.3 (Pin_3), J17.3 (Pin_3)
- new net: J15.4 (Pin_4), J17.4 (Pin_4)
- new net: J15.5 (Pin_5), J17.5 (Pin_5)
- new net: J15.6 (Pin_6), J17.6 (Pin_6)
- new net: J15.7 (Pin_7), J17.7 (Pin_7)
- new net: J16.1 (Pin_1), J18.1 (Pin_1)
- new net: J16.10 (Pin_10), J18.10 (Pin_10)
- new net: J16.11 (Pin_11), J18.11 (Pin_11)
- new net: J16.15 (Pin_15), J18.15 (Pin_15)
- new net: J16.2 (Pin_2), J18.2 (Pin_2)
- new net: J16.3 (Pin_3), J18.3 (Pin_3)
- new net: J16.4 (Pin_4), J18.4 (Pin_4)
- new net: J16.5 (Pin_5), J18.5 (Pin_5)
- new net: J16.7 (Pin_7), J18.7 (Pin_7)
- new net BT_RX: J5.2 (Pin_2), R6.2, R7.1
- no-connect marks 32 -> 23
Other:
- note added: "*D10"
- note added: "*D11"
- note added: "*D3"
- note added: "*D5"
- note added: "*D6"
- note added: "*D9"
- note added: "3.3V"
- note added: "A0"
- note added: "A1"
- note added: "A2"
- note added: "A3"
- note added: "A4"
- note added: "A5"
- note added: "A6"
- note added: "A7"
- note added: "BLUETOOTH"
- note added: "D12"
- note added: "D13"
- note added: "D2"
- note added: "D4"
- note added: "D7"
- note added: "D8"
- note added: "GPS"
- note added: "MAGNETOMETER"
- note added: "REF"
- note added: "RST"
- note added: "RX0"
- note added: "|_________________| RIBBON CABLE"
- note removed: "PROG PINS"
- note removed: "RST BTN"
- moved on the sheet: J1, J2, J3

Commit message: SanBan Rev 1.0
Parts:
- J1, J2: footprint Connector_PinSocket_2.54mm:PinSocket_1x12_P2.54mm_Vertical -> Connector_PinSocket_2.00mm:PinSocket_1x12_P2.00mm_Vertical
- J10, J11, J6, J7, J8, J9: footprint Connector_PinHeader_2.54mm:PinHeader_1x03_P2.54mm_Horizontal -> Connector_PinHeader_2.54mm:PinHeader_1x03_P2.54mm_Vertical
- J3: footprint Connector_PinSocket_2.00mm:PinSocket_1x09_P2.00mm_Vertical -> Connector_PinSocket_2.54mm:PinSocket_1x09_P2.54mm_Vertical
- J4: footprint Connector_Wire:SolderWire-0.127sqmm_1x02_P3.7mm_D0.48mm_OD1mm -> Connector_PinHeader_2.54mm:PinHeader_1x02_P2.54mm_Horizontal
Changed lines of the file:
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@@
       (effects (font (size 1.27 1.27)))
     )
-    (property "Footprint" "Connector_PinHeader_2.54mm:PinHeader_1x03_P2.54mm_Horizontal" (at 72.39 88.9 0)
+    (property "Footprint" "Connector_PinHeader_2.54mm:PinHeader_1x03_P2.54mm_Vertical" (at 72.39 88.9 0)
       (effects (font (size 1.27 1.27)) hide)
     )
@@
       (effects (font (size 1.27 1.27)))
     )
-    (property "Footprint" "Connector_PinHeader_2.54mm:PinHeader_1x03_P2.54mm_Horizontal" (at 72.39 107.95 0)
+    (property "Footprint" "Connector_PinHeader_2.54mm:PinHeader_1x03_P2.54mm_Vertical" (at 72.39 107.95 0)
       (effects (font (size 1.27 1.27)) hide)
     )
@@
       (effects (font (size 1.27 1.27)) (justify right))
     )
-    (property "Footprint" "Connector_PinSocket_2.54mm:PinSocket_1x12_P2.54mm_Vertical" (at 184.15 105.41 0)
+    (property "Footprint" "Connector_PinSocket_2.00mm:PinSocket_1x12_P2.00mm_Vertical" (at 184.15 105.41 0)
       (effects (font (size 1.27 1.27)) hide)
     )
@@
       (effects (font (size 1.27 1.27)))
     )
-    (property "Footprint" "Connector_PinHeader_2.54mm:PinHeader_1x03_P2.54mm_Horizontal" (at 45.72 107.95 0)
+    (property "Footprint" "Connector_PinHeader_2.54mm:PinHeader_1x03_P2.54mm_Vertical" (at 45.72 107.95 0)
       (effects (font (size 1.27 1.27)) hide)
     )
@@
       (effects (font (size 1.27 1.27)))
     )
-    (property "Footprint" "Connector_PinSocket_2.00mm:PinSocket_1x09_P2.00mm_Vertical" (at 219.71 107.95 0)
+    (property "Footprint" "Connector_PinSocket_2.54mm:PinSocket_1x09_P2.54mm_Vertical" (at 219.71 107.95 0)
       (effects (font (size 1.27 1.27)) hide)
     )
@@
       (effects (font (size 1.27 1.27)))
     )
-    (property "Footprint" "Connector_PinHeader_2.54mm:PinHeader_1x03_P2.54mm_Horizontal" (at 45.72 88.9 0)
+    (property "Footprint" "Connector_PinHeader_2.54mm:PinHeader_1x03_P2.54mm_Vertical" (at 45.72 88.9 0)
       (effects (font (size 1.27 1.27)) hide)
     )
@@
       (effects (font (size 1.27 1.27)))
     )
-    (property "Footprint" "Connector_PinSocket_2.54mm:PinSocket_1x12_P2.54mm_Vertical" (at 203.2 124.46 0)
+    (property "Footprint" "Connector_PinSocket_2.00mm:PinSocket_1x12_P2.00mm_Vertical" (at 203.2 124.46 0)
       (effects (font (size 1.27 1.27)) hide)
     )
@@
       (effects (font (size 1.27 1.27)))
     )
-    (property "Footprint" "Connector_PinHeader_2.54mm:PinHeader_1x03_P2.54mm_Horizontal" (at 99.06 88.9 0)
+    (property "Footprint" "Connector_PinHeader_2.54mm:PinHeader_1x03_P2.54mm_Vertical" (at 99.06 88.9 0)
       (effects (font (size 1.27 1.27)) hide)
     )
@@
       (effects (font (size 1.27 1.27)))
     )
-    (property "Footprint" "Connector_PinHeader_2.54mm:PinHeader_1x03_P2.54mm_Horizontal" (at 99.06 107.95 0)
+    (property "Footprint" "Connector_PinHeader_2.54mm:PinHeader_1x03_P2.54mm_Vertical" (at 99.06 107.95 0)
       (effects (font (size 1.27 1.27)) hide)
     )
@@
       (effects (font (size 1.27 1.27)))
     )
-    (property "Footprint" "Connector_Wire:SolderWire-0.127sqmm_1x02_P3.7mm_D0.48mm_OD1mm" (at 115.57 26.67 0)
-      (effects (font (size 1.27 1.27)) hide)
-    )
+    (property "Footprint" "Connector_PinHeader_2.54mm:PinHeader_1x02_P2.54mm_Horizontal" (at 115.57 26.67 0)
+      (effects (font (size 1.27 1.27)) hide)
+    )

Commit message: Submitted Rev 1 SanBan
Parts:
- added JP1, JP2: SolderJumper_2_Open, Jumper:SolderJumper-2_P1.3mm_Open_RoundedPad1.0x1.5mm, symbol Jumper:SolderJumper_2_Open
- added R4: 20K, Capacitor_SMD:C_0805_2012Metric_Pad1.18x1.45mm_HandSolder, symbol Device:R
- added R5: 2K, Capacitor_SMD:C_0805_2012Metric_Pad1.18x1.45mm_HandSolder, symbol Device:R
- R2: value 115k -> 33K
- R3: value 22.1k -> 82K
- renumbered R4 to R6, R6 to R7, R7 to R8
Connections:
- net +5V: now also JP1.2 (B)
- net GND: now also JP2.1 (A), R5.1; no longer R3.2
- net at C3.1, IC1.5 (FB), R3.1: now also R4.1; no longer R2.2
- new net: JP2.2 (B), R4.2, R5.2
- new net: JP1.1 (A), R2.2, R3.2
Other:
- note added: "R2+R3 = 115K NOMINAL R +R = 22.1K NOMINAL"
- moved on the sheet: C1, J1, J15, J16, J17, J18, J2, J3, R2, R3, R7, R8
